File: PCB/0.1/Orthonite87_PCB.kicad_pcb (KiCad board)
At the start: 2 copper layers, 0 parts

Commit message: Schematic update
Near finished with rev0.1
Parts:
- added BZ1: Buzzer, Buzzer_Beeper:Buzzer_Murata_PKMCS0909E4000-R1, B.Cu at (151.6, 81.0)
- added C1: 4u7, Capacitor_SMD:C_0603_1608Metric, B.Cu at (98.8, 76.8)
- added C10: 15p, Capacitor_SMD:C_0603_1608Metric, B.Cu at (124.5, 82.0)
- added C11: 15p, Capacitor_SMD:C_0603_1608Metric, B.Cu at (123.6, 76.2)
- added C12: 4u7, Capacitor_SMD:C_0603_1608Metric, B.Cu at (40.5, 59.5)
- added C13: 10u, Capacitor_SMD:C_0603_1608Metric, B.Cu at (35.8, 62.7)
- added C14: 100n, Capacitor_SMD:C_0603_1608Metric, B.Cu at (74.9, 58.0)
- added C15: 100n, Capacitor_SMD:C_0603_1608Metric, B.Cu at (132.0, 58.2)
- added C16: 100n, Capacitor_SMD:C_0603_1608Metric, B.Cu at (179.7, 58.2)
- added C17: 100n, Capacitor_SMD:C_0603_1608Metric, B.Cu at (246.3, 58.2)
- added C18: 100n, Capacitor_SMD:C_0603_1608Metric, B.Cu at (303.5, 58.2)
- added C19: 100n, Capacitor_SMD:C_0603_1608Metric, B.Cu at (303.4, 77.2)
- added C2: 100n, Capacitor_SMD:C_0603_1608Metric, B.Cu at (112.4, 70.1)
- added C20: 100n, Capacitor_SMD:C_0603_1608Metric, B.Cu at (246.4, 77.2)
- added C21: 100n, Capacitor_SMD:C_0603_1608Metric, B.Cu at (179.7, 77.2)
- added C22: 100n, Capacitor_SMD:C_0603_1608Metric, B.Cu at (132.1, 77.2)
- added C23: 100n, Capacitor_SMD:C_0603_1608Metric, B.Cu at (74.9, 77.2)
- added C24: 100n, Capacitor_SMD:C_0603_1608Metric, B.Cu at (74.9, 96.3)
- added C25: 100n, Capacitor_SMD:C_0603_1608Metric, B.Cu at (132.1, 96.3)
- added C26: 100n, Capacitor_SMD:C_0603_1608Metric, B.Cu at (179.7, 96.3)
- added C27: 100n, Capacitor_SMD:C_0603_1608Metric, B.Cu at (246.5, 96.3)
- added C28: 100n, Capacitor_SMD:C_0603_1608Metric, B.Cu at (303.5, 96.3)
- added C29: 100n, Capacitor_SMD:C_0603_1608Metric, B.Cu at (303.7, 115.3)
- added C3: 100n, Capacitor_SMD:C_0603_1608Metric, B.Cu at (101.3, 75.9)
- added C30: 100n, Capacitor_SMD:C_0603_1608Metric, B.Cu at (221.0, 115.3)
- added C31: 100n, Capacitor_SMD:C_0603_1608Metric, B.Cu at (179.7, 115.3)
- added C32: 100n, Capacitor_SMD:C_0603_1608Metric, B.Cu at (141.7, 115.3)
- added C33: 100n, Capacitor_SMD:C_0603_1608Metric, B.Cu at (94.1, 115.3)
- added C34: 100n, Capacitor_SMD:C_0603_1608Metric, B.Cu at (74.3, 128.3)
- added C35: 100n, Capacitor_SMD:C_0603_1608Metric, B.Cu at (131.4, 128.1)
- added C36: 100n, Capacitor_SMD:C_0603_1608Metric, B.Cu at (226.6, 128.3)
- added C37: 100n, Capacitor_SMD:C_0603_1608Metric, B.Cu at (283.7, 128.5)
- added C4: 100n, Capacitor_SMD:C_0603_1608Metric, B.Cu at (109.1, 89.0)
- added C5: 100n, Capacitor_SMD:C_0603_1608Metric, B.Cu at (118.7, 84.6)
- added C6: 100n, Capacitor_SMD:C_0603_1608Metric, B.Cu at (112.9, 89.2)
- added C7: 10u, Capacitor_SMD:C_0603_1608Metric, B.Cu at (27.8, 46.8)
- added C8: 1u, Capacitor_SMD:C_0603_1608Metric, B.Cu at (88.9, 61.9)
- added C9: 1u, Capacitor_SMD:C_0603_1608Metric, B.Cu at (95.2, 61.9)
- added D1: WS2812B, LED_SMD:LED_WS2812B_PLCC4_5.0x5.0mm_P3.2mm, B.Cu at (73.0, 61.9)
- added D10: WS2812B, LED_SMD:LED_WS2812B_PLCC4_5.0x5.0mm_P3.2mm, B.Cu at (73.0, 81.0)
- added D11: WS2812B, LED_SMD:LED_WS2812B_PLCC4_5.0x5.0mm_P3.2mm, B.Cu at (73.0, 100.0)
- added D12: WS2812B, LED_SMD:LED_WS2812B_PLCC4_5.0x5.0mm_P3.2mm, B.Cu at (130.2, 100.0)
- added D13: WS2812B, LED_SMD:LED_WS2812B_PLCC4_5.0x5.0mm_P3.2mm, B.Cu at (177.8, 100.0)
- added D14: WS2812B, LED_SMD:LED_WS2812B_PLCC4_5.0x5.0mm_P3.2mm, B.Cu at (244.5, 100.0)
- added D15: WS2812B, LED_SMD:LED_WS2812B_PLCC4_5.0x5.0mm_P3.2mm, B.Cu at (301.6, 100.0)
- added D16: WS2812B, LED_SMD:LED_WS2812B_PLCC4_5.0x5.0mm_P3.2mm, B.Cu at (301.6, 119.1)
- added D17: WS2812B, LED_SMD:LED_WS2812B_PLCC4_5.0x5.0mm_P3.2mm, B.Cu at (219.1, 119.1)
- added D18: WS2812B, LED_SMD:LED_WS2812B_PLCC4_5.0x5.0mm_P3.2mm, B.Cu at (177.8, 119.1)
- added D19: WS2812B, LED_SMD:LED_WS2812B_PLCC4_5.0x5.0mm_P3.2mm, B.Cu at (139.7, 119.1)
- added D2: WS2812B, LED_SMD:LED_WS2812B_PLCC4_5.0x5.0mm_P3.2mm, B.Cu at (130.2, 61.9)
- added D20: WS2812B, LED_SMD:LED_WS2812B_PLCC4_5.0x5.0mm_P3.2mm, B.Cu at (92.1, 119.1)
- added D21: SK6812-MINI-E, josh-led:SK8612-MINI-E, F.Cu at (75.1, 122.6)
- added D22: SK6812-MINI-E, josh-led:SK8612-MINI-E, F.Cu at (132.1, 122.5)
- added D23: SK6812-MINI-E, josh-led:SK8612-MINI-E, F.Cu at (227.3, 122.6)
- added D24: SK6812-MINI-E, josh-led:SK8612-MINI-E, F.Cu at (284.4, 122.7)
- added D25: LE_RED, josh-led:LED_0603_1608Metric_45_noSilk, B.Cu at (14.3, 44.5)
- added D26: 1N4148, Diode_SMD:D_SOD-123, B.Cu at (38.9, 62.7)
- added D3: WS2812B, LED_SMD:LED_WS2812B_PLCC4_5.0x5.0mm_P3.2mm, B.Cu at (177.8, 61.9)
- added D4: WS2812B, LED_SMD:LED_WS2812B_PLCC4_5.0x5.0mm_P3.2mm, B.Cu at (244.5, 61.9)
- added D5: WS2812B, LED_SMD:LED_WS2812B_PLCC4_5.0x5.0mm_P3.2mm, B.Cu at (301.6, 61.9)
- added D6: WS2812B, LED_SMD:LED_WS2812B_PLCC4_5.0x5.0mm_P3.2mm, B.Cu at (301.6, 81.0)
- added D7: WS2812B, LED_SMD:LED_WS2812B_PLCC4_5.0x5.0mm_P3.2mm, B.Cu at (244.5, 81.0)
- added D8: WS2812B, LED_SMD:LED_WS2812B_PLCC4_5.0x5.0mm_P3.2mm, B.Cu at (177.8, 81.0)
- added D9: WS2812B, LED_SMD:LED_WS2812B_PLCC4_5.0x5.0mm_P3.2mm, B.Cu at (130.2, 81.0)
- added D_1: 1N4148, Diode_SMD:D_SOD-123, B.Cu at (33.4, 33.7)
- added D_10: 1N4148, Diode_SMD:D_SOD-123, B.Cu at (204.9, 33.6)
- added D_100: 1N4148, Diode_SMD:D_SOD-123, B.Cu at (322.3, 128.2)
- added D_11: 1N4148, Diode_SMD:D_SOD-123, B.Cu at (223.9, 33.6)
- added D_12: 1N4148, Diode_SMD:D_SOD-123, B.Cu at (243.0, 33.6)
- added D_13: 1N4148, Diode_SMD:D_SOD-123, B.Cu at (262.0, 33.6)
- added D_14: 1N4148, Diode_SMD:D_SOD-123, B.Cu at (281.1, 33.6)
- added D_15: 1N4148, Diode_SMD:D_SOD-123, B.Cu at (300.1, 33.6)
- added D_16: 1N4148, Diode_SMD:D_SOD-123, B.Cu at (303.1, 33.6)
- added D_17: 1N4148, Diode_SMD:D_SOD-123, B.Cu at (52.5, 52.7)
- added D_18: 1N4148, Diode_SMD:D_SOD-123, B.Cu at (71.5, 52.7)
- added D_19: 1N4148, Diode_SMD:D_SOD-123, B.Cu at (90.6, 52.6)
- added D_2: 1N4148, Diode_SMD:D_SOD-123, B.Cu at (52.5, 33.7)
- added D_20: 1N4148, Diode_SMD:D_SOD-123, B.Cu at (109.6, 52.7)
- added D_21: 1N4148, Diode_SMD:D_SOD-123, B.Cu at (128.7, 52.6)
- added D_22: 1N4148, Diode_SMD:D_SOD-123, B.Cu at (147.7, 52.6)
- added D_23: 1N4148, Diode_SMD:D_SOD-123, B.Cu at (166.8, 52.6)
- added D_24: 1N4148, Diode_SMD:D_SOD-123, B.Cu at (185.8, 52.7)
- added D_25: 1N4148, Diode_SMD:D_SOD-123, B.Cu at (204.9, 52.7)
- added D_26: 1N4148, Diode_SMD:D_SOD-123, B.Cu at (223.9, 52.6)
- added D_27: 1N4148, Diode_SMD:D_SOD-123, B.Cu at (243.0, 52.7)
- added D_28: 1N4148, Diode_SMD:D_SOD-123, B.Cu at (262.0, 52.6)
- added D_29: 1N4148, Diode_SMD:D_SOD-123, B.Cu at (281.1, 52.6)
- added D_3: 1N4148, Diode_SMD:D_SOD-123, B.Cu at (71.4, 33.6)
- added D_30: 1N4148, Diode_SMD:D_SOD-123, B.Cu at (300.1, 52.6)
- added D_31: 1N4148, Diode_SMD:D_SOD-123, B.Cu at (303.1, 52.6)
- added D_32: 1N4148, Diode_SMD:D_SOD-123, B.Cu at (319.2, 45.2)
- added D_33: 1N4148, Diode_SMD:D_SOD-123, B.Cu at (33.4, 71.1)
- added D_34: 1N4148, Diode_SMD:D_SOD-123, B.Cu at (52.5, 64.3)
- added D_35: 1N4148, Diode_SMD:D_SOD-123, B.Cu at (71.5, 71.1)
- added D_36: 1N4148, Diode_SMD:D_SOD-123, B.Cu at (90.6, 71.1)
- added D_37: 1N4148, Diode_SMD:D_SOD-123, B.Cu at (93.7, 71.1)
- added D_38: 1N4148, Diode_SMD:D_SOD-123, B.Cu at (128.7, 71.1)
- added D_39: 1N4148, Diode_SMD:D_SOD-123, B.Cu at (147.7, 71.1)
- added D_4: 1N4148, Diode_SMD:D_SOD-123, B.Cu at (90.5, 33.6)
- added D_40: 1N4148, Diode_SMD:D_SOD-123, B.Cu at (166.8, 71.1)
- added D_41: 1N4148, Diode_SMD:D_SOD-123, B.Cu at (185.8, 71.1)
- added D_42: 1N4148, Diode_SMD:D_SOD-123, B.Cu at (204.9, 71.1)
- added D_43: 1N4148, Diode_SMD:D_SOD-123, B.Cu at (223.9, 71.1)
- added D_44: 1N4148, Diode_SMD:D_SOD-123, B.Cu at (243.0, 71.1)
- added D_45: 1N4148, Diode_SMD:D_SOD-123, B.Cu at (262.0, 71.1)
- added D_46: 1N4148, Diode_SMD:D_SOD-123, B.Cu at (281.1, 71.1)
- added D_47: 1N4148, Diode_SMD:D_SOD-123, B.Cu at (300.1, 71.1)
- added D_48: 1N4148, Diode_SMD:D_SOD-123, B.Cu at (319.2, 71.1)
- added D_49: 1N4148, Diode_SMD:D_SOD-123, B.Cu at (322.2, 71.1)
- added D_5: 1N4148, Diode_SMD:D_SOD-123, B.Cu at (109.6, 34.2)
- added D_50: 1N4148, Diode_SMD:D_SOD-123, B.Cu at (33.4, 90.1)
- added D_51: 1N4148, Diode_SMD:D_SOD-123, B.Cu at (52.5, 83.4)
- added D_52: 1N4148, Diode_SMD:D_SOD-123, B.Cu at (71.5, 89.5)
- added D_53: 1N4148, Diode_SMD:D_SOD-123, B.Cu at (90.6, 90.1)
- added D_54: 1N4148, Diode_SMD:D_SOD-123, B.Cu at (93.7, 90.1)
- added D_55: 1N4148, Diode_SMD:D_SOD-123, B.Cu at (128.7, 90.1)
- added D_56: 1N4148, Diode_SMD:D_SOD-123, B.Cu at (147.7, 90.1)
- added D_57: 1N4148, Diode_SMD:D_SOD-123, B.Cu at (166.8, 90.1)
- added D_58: 1N4148, Diode_SMD:D_SOD-123, B.Cu at (185.8, 90.2)
- added D_59: 1N4148, Diode_SMD:D_SOD-123, B.Cu at (204.9, 90.1)
- added D_6: 1N4148, Diode_SMD:D_SOD-123, B.Cu at (128.7, 33.6)
- added D_60: 1N4148, Diode_SMD:D_SOD-123, B.Cu at (223.9, 90.1)
- added D_61: 1N4148, Diode_SMD:D_SOD-123, B.Cu at (242.9, 90.1)
- added D_62: 1N4148, Diode_SMD:D_SOD-123, B.Cu at (262.0, 90.1)
- added D_63: 1N4148, Diode_SMD:D_SOD-123, B.Cu at (281.1, 90.1)
- added D_64: 1N4148, Diode_SMD:D_SOD-123, B.Cu at (300.1, 90.1)
- added D_65: 1N4148, Diode_SMD:D_SOD-123, B.Cu at (303.1, 90.1)
- added D_66: 1N4148, Diode_SMD:D_SOD-123, B.Cu at (319.2, 83.3)
- added D_67: 1N4148, Diode_SMD:D_SOD-123, B.Cu at (33.3, 109.2)
- added D_68: 1N4148, Diode_SMD:D_SOD-123, B.Cu at (52.5, 102.4)
- added D_69: 1N4148, Diode_SMD:D_SOD-123, B.Cu at (71.5, 109.2)
- added D_7: 1N4148, Diode_SMD:D_SOD-123, B.Cu at (147.7, 33.6)
- added D_70: 1N4148, Diode_SMD:D_SOD-123, B.Cu at (90.5, 109.2)
- added D_71: 1N4148, Diode_SMD:D_SOD-123, B.Cu at (109.5, 109.2)
- added D_72: 1N4148, Diode_SMD:D_SOD-123, B.Cu at (128.6, 109.2)
- added D_73: 1N4148, Diode_SMD:D_SOD-123, B.Cu at (147.6, 109.2)
- added D_74: 1N4148, Diode_SMD:D_SOD-123, B.Cu at (166.7, 109.2)
- added D_75: 1N4148, Diode_SMD:D_SOD-123, B.Cu at (185.7, 109.2)
- added D_76: 1N4148, Diode_SMD:D_SOD-123, B.Cu at (204.8, 109.2)
- added D_77: 1N4148, Diode_SMD:D_SOD-123, B.Cu at (223.8, 109.2)
- added D_78: 1N4148, Diode_SMD:D_SOD-123, B.Cu at (242.9, 109.2)
- added D_79: 1N4148, Diode_SMD:D_SOD-123, B.Cu at (261.9, 109.2)
- added D_8: 1N4148, Diode_SMD:D_SOD-123, B.Cu at (166.8, 33.6)
- added D_80: 1N4148, Diode_SMD:D_SOD-123, B.Cu at (281.0, 109.2)
- added D_81: 1N4148, Diode_SMD:D_SOD-123, B.Cu at (300.0, 109.2)
- added D_82: 1N4148, Diode_SMD:D_SOD-123, B.Cu at (303.2, 109.2)
- added D_83: 1N4148, Diode_SMD:D_SOD-123, B.Cu at (319.1, 102.4)
- added D_84: 1N4148, Diode_SMD:D_SOD-123, B.Cu at (33.3, 128.3)
- added D_85: 1N4148, Diode_SMD:D_SOD-123, B.Cu at (52.4, 128.3)
- added D_86: 1N4148, Diode_SMD:D_SOD-123, B.Cu at (71.4, 128.2)
- added D_87: 1N4148, Diode_SMD:D_SOD-123, B.Cu at (90.5, 128.3)
- added D_88: 1N4148, Diode_SMD:D_SOD-123, B.Cu at (109.5, 128.2)
- added D_89: 1N4148, Diode_SMD:D_SOD-123, B.Cu at (128.6, 128.2)
- added D_9: 1N4148, Diode_SMD:D_SOD-123, B.Cu at (185.8, 33.6)
- added D_90: 1N4148, Diode_SMD:D_SOD-123, B.Cu at (147.6, 128.3)
- added D_91: 1N4148, Diode_SMD:D_SOD-123, B.Cu at (166.8, 128.2)
- added D_92: 1N4148, Diode_SMD:D_SOD-123, B.Cu at (185.8, 128.2)
- added D_93: 1N4148, Diode_SMD:D_SOD-123, B.Cu at (204.8, 128.2)
- added D_94: 1N4148, Diode_SMD:D_SOD-123, B.Cu at (223.8, 128.2)
- added D_95: 1N4148, Diode_SMD:D_SOD-123, B.Cu at (243.0, 128.2)
- added D_96: 1N4148, Diode_SMD:D_SOD-123, B.Cu at (261.9, 128.2)
- added D_97: 1N4148, Diode_SMD:D_SOD-123, B.Cu at (281.0, 128.2)
- added D_98: 1N4148, Diode_SMD:D_SOD-123, B.Cu at (300.1, 128.2)
- added D_99: 1N4148, Diode_SMD:D_SOD-123, B.Cu at (319.1, 128.2)
- added F1: 500mA, josh-passives-smt:Fuse_0805_2012Metric, B.Cu at (30.3, 47.6)
- added J1: USB_C_U262-161N-4BVC11, josh-connectors:USB_C_U262-161N-4BVC11, B.Cu at (10.3, 52.4)
- added J2: SWD, josh-connectors:STM_4_PIN_THT_Staggered, B.Cu at (34.9, 48.4)
- added K_1: 0,15, josh-keyboard:MX_KEYSWITCH_ENCODER, F.Cu at (311.1, 33.3)
- added K_10: 0,8, josh-keyboard:MXOnly-1U-NoLED, F.Cu at (177.8, 33.3)
- added K_100: 5,9, josh-keyboard:MXOnly-1U-NoLED, F.Cu at (177.8, 128.6)
- added K_101: 5,10, josh-keyboard:MXOnly-1U-NoLED, F.Cu at (196.8, 128.6)
- added K_102: 5,11, josh-keyboard:MXOnly-1U-NoLED, F.Cu at (215.9, 128.6)
- added K_103: 5,12, josh-keyboard:MXOnly-1U-NoLED, F.Cu at (234.9, 128.6)
- added K_104: 5,14, josh-keyboard:MXOnly-3U-ReversedStabilizers-NoLED, F.Cu at (254.0, 128.6)
- added K_105: 5,15, josh-keyboard:MXOnly-1U-NoLED, F.Cu at (273.1, 128.6)
- added K_106: 5,16, josh-keyboard:MXOnly-1U-NoLED, F.Cu at (292.1, 128.6)
- added K_107: 5,17, josh-keyboard:MXOnly-1U-NoLED, F.Cu at (311.1, 128.6)
- added K_108: 5,18, josh-keyboard:MXOnly-1U-NoLED, F.Cu at (330.2, 128.6)
- added K_11: 0,9, josh-keyboard:MXOnly-1U-NoLED, F.Cu at (196.8, 33.3)
- added K_12: 0,10, josh-keyboard:MXOnly-1U-NoLED, F.Cu at (215.9, 33.3)
- added K_13: 0,11, josh-keyboard:MXOnly-1U-NoLED, F.Cu at (234.9, 33.3)
- added K_14: 0,12, josh-keyboard:MXOnly-1U-NoLED, F.Cu at (254.0, 33.3)
- added K_15: 0,13, josh-keyboard:MXOnly-1U-NoLED, F.Cu at (273.1, 33.3)
- added K_16: 0,14, josh-keyboard:MXOnly-1U-NoLED, F.Cu at (292.1, 33.3)
- added K_17: 1,15, josh-keyboard:MXOnly-1U-NoLED, F.Cu at (311.1, 52.4)
- added K_18: 1,1, josh-keyboard:MXOnly-1U-NoLED, F.Cu at (44.5, 52.4)
- added K_19: 1,2, josh-keyboard:MXOnly-1U-NoLED, F.Cu at (63.5, 52.4)
- added K_2: 0,0, josh-keyboard:MXOnly-1U-NoLED, F.Cu at (25.4, 33.3)
- added K_20: 1,3, josh-keyboard:MXOnly-1U-NoLED, F.Cu at (82.5, 52.4)
- added K_21: 1,4, josh-keyboard:MXOnly-1U-NoLED, F.Cu at (101.6, 52.4)
- added K_22: 1,5, josh-keyboard:MXOnly-1U-NoLED, F.Cu at (120.7, 52.4)
- added K_23: 1,6, josh-keyboard:MXOnly-1U-NoLED, F.Cu at (139.7, 52.4)
- added K_24: 1,7, josh-keyboard:MXOnly-1U-NoLED, F.Cu at (158.8, 52.4)
- added K_25: 1,8, josh-keyboard:MXOnly-1U-NoLED, F.Cu at (177.8, 52.4)
- added K_26: 1,9, josh-keyboard:MXOnly-1U-NoLED, F.Cu at (196.8, 52.4)
- added K_27: 1,10, josh-keyboard:MXOnly-1U-NoLED, F.Cu at (215.9, 52.4)
- added K_28: 1,11, josh-keyboard:MXOnly-1U-NoLED, F.Cu at (234.9, 52.4)
- added K_29: 1,12, josh-keyboard:MXOnly-1U-NoLED, F.Cu at (254.0, 52.4)
- added K_3: 0,1, josh-keyboard:MXOnly-1U-NoLED, F.Cu at (44.5, 33.3)
- added K_30: 1,13, josh-keyboard:MXOnly-1U-NoLED, F.Cu at (273.1, 52.4)
- added K_31: 1,14, josh-keyboard:MXOnly-1U-NoLED, F.Cu at (292.1, 52.4)
- added K_32: 1,16, josh-keyboard:MXOnly-2U-NoLED, F.Cu at (320.7, 52.4)
- added K_33: 1,17, josh-keyboard:MXOnly-1U-NoLED, F.Cu at (330.2, 52.4)
- added K_34: 2,1, josh-keyboard:MXOnly-1U-NoLED, F.Cu at (44.5, 71.4)
- added K_35: 2,0, josh-keyboard:MXOnly-1U-NoLED, F.Cu at (25.4, 71.4)
- added K_36: 2,2, josh-keyboard:MXOnly-2U-NoLED, F.Cu at (54.0, 71.4)
- added K_37: 2,3, josh-keyboard:MXOnly-1U-NoLED, F.Cu at (63.5, 71.4)
- added K_38: 2,4, josh-keyboard:MXOnly-1U-NoLED, F.Cu at (82.5, 71.4)
- added K_39: 2,5, josh-keyboard:MXOnly-1U-NoLED, F.Cu at (101.6, 71.4)
- added K_4: 0,2, josh-keyboard:MXOnly-1U-NoLED, F.Cu at (63.5, 33.3)
- added K_40: 2,6, josh-keyboard:MXOnly-1U-NoLED, F.Cu at (120.7, 71.4)
- added K_41: 2,7, josh-keyboard:MXOnly-1U-NoLED, F.Cu at (139.7, 71.4)
- added K_42: 2,8, josh-keyboard:MXOnly-1U-NoLED, F.Cu at (158.8, 71.4)
- added K_43: 2,9, josh-keyboard:MXOnly-1U-NoLED, F.Cu at (177.8, 71.4)
- added K_44: 2,10, josh-keyboard:MXOnly-1U-NoLED, F.Cu at (196.8, 71.4)
- added K_45: 2,11, josh-keyboard:MXOnly-1U-NoLED, F.Cu at (215.9, 71.4)
- added K_46: 2,12, josh-keyboard:MXOnly-1U-NoLED, F.Cu at (234.9, 71.4)
- added K_47: 2,13, josh-keyboard:MXOnly-1U-NoLED, F.Cu at (254.0, 71.4)
- added K_48: 2,14, josh-keyboard:MXOnly-1U-NoLED, F.Cu at (273.1, 71.4)
- added K_49: 2,15, josh-keyboard:MXOnly-1U-NoLED, F.Cu at (292.1, 71.4)
- added K_5: 0,3, josh-keyboard:MXOnly-1U-NoLED, F.Cu at (82.5, 33.3)
- added K_50: 2,16, josh-keyboard:MXOnly-1U-NoLED, F.Cu at (311.1, 71.4)
- added K_51: 2,17, josh-keyboard:MXOnly-1U-NoLED, F.Cu at (330.2, 71.4)
- added K_52: 3,1, josh-keyboard:MXOnly-1U-NoLED, F.Cu at (44.5, 90.5)
- added K_53: 3,17, josh-keyboard:MXOnly-1U-NoLED, F.Cu at (330.2, 90.5)
- added K_54: 3,0, josh-keyboard:MXOnly-1U-NoLED, F.Cu at (25.4, 90.5)
- added K_55: 3,2, josh-keyboard:MXOnly-2U-NoLED, F.Cu at (54.0, 90.5)
- added K_56: 3,3, josh-keyboard:MXOnly-1U-NoLED, F.Cu at (63.5, 90.5)
- added K_57: 3,4, josh-keyboard:MXOnly-1U-NoLED, F.Cu at (82.5, 90.5)
- added K_58: 3,5, josh-keyboard:MXOnly-1U-NoLED, F.Cu at (101.6, 90.5)
- added K_59: 3,6, josh-keyboard:MXOnly-1U-NoLED, F.Cu at (120.7, 90.5)
- added K_6: 0,4, josh-keyboard:MXOnly-1U-NoLED, F.Cu at (101.6, 33.3)
- added K_60: 3,7, josh-keyboard:MXOnly-1U-NoLED, F.Cu at (139.7, 90.5)
- added K_61: 3,8, josh-keyboard:MXOnly-1U-NoLED, F.Cu at (158.8, 90.5)
- added K_62: 3,9, josh-keyboard:MXOnly-1U-NoLED, F.Cu at (177.8, 90.5)
- added K_63: 3,10, josh-keyboard:MXOnly-1U-NoLED, F.Cu at (196.8, 90.5)
- added K_64: 3,11, josh-keyboard:MXOnly-1U-NoLED, F.Cu at (215.9, 90.5)
- added K_65: 3,12, josh-keyboard:MXOnly-1U-NoLED, F.Cu at (234.9, 90.5)
- added K_66: 3,13, josh-keyboard:MXOnly-1U-NoLED, F.Cu at (254.0, 90.5)
- added K_67: 3,14, josh-keyboard:MXOnly-1U-NoLED, F.Cu at (273.1, 90.5)
- added K_68: 3,15, josh-keyboard:MXOnly-1U-NoLED, F.Cu at (292.1, 90.5)
- added K_69: 3,16, josh-keyboard:MXOnly-1U-NoLED, F.Cu at (311.1, 90.5)
- added K_7: 0,5, josh-keyboard:MXOnly-1U-NoLED, F.Cu at (120.7, 33.3)
- added K_70: 3,18, josh-keyboard:MXOnly-2U-NoLED, F.Cu at (320.7, 90.5)
- added K_71: 4,1, josh-keyboard:MXOnly-1U-NoLED, F.Cu at (44.5, 109.5)
- added K_72: 4,17, josh-keyboard:MXOnly-1U-NoLED, F.Cu at (330.2, 109.5)
- added K_73: 4,0, josh-keyboard:MXOnly-1U-NoLED, F.Cu at (25.4, 109.5)
- added K_74: 4,2, josh-keyboard:MXOnly-2U-NoLED, F.Cu at (54.0, 109.5)
- added K_75: 4,3, josh-keyboard:MXOnly-1U-NoLED, F.Cu at (63.5, 109.5)
- added K_76: 4,4, josh-keyboard:MXOnly-1U-NoLED, F.Cu at (82.5, 109.5)
- added K_77: 4,5, josh-keyboard:MXOnly-1U-NoLED, F.Cu at (101.6, 109.5)
- added K_78: 4,6, josh-keyboard:MXOnly-1U-NoLED, F.Cu at (120.7, 109.5)
- added K_79: 4,7, josh-keyboard:MXOnly-1U-NoLED, F.Cu at (139.7, 109.5)
- added K_8: 0,6, josh-keyboard:MXOnly-1U-NoLED, F.Cu at (139.7, 33.3)
- added K_80: 4,8, josh-keyboard:MXOnly-1U-NoLED, F.Cu at (158.8, 109.5)
- added K_81: 4,9, josh-keyboard:MXOnly-1U-NoLED, F.Cu at (177.8, 109.5)
- added K_82: 4,10, josh-keyboard:MXOnly-1U-NoLED, F.Cu at (196.8, 109.5)
- added K_83: 4,11, josh-keyboard:MXOnly-1U-NoLED, F.Cu at (215.9, 109.5)
- added K_84: 4,12, josh-keyboard:MXOnly-1U-NoLED, F.Cu at (234.9, 109.5)
- added K_85: 4,13, josh-keyboard:MXOnly-1U-NoLED, F.Cu at (254.0, 109.5)
- added K_86: 4,14, josh-keyboard:MXOnly-1U-NoLED, F.Cu at (273.1, 109.5)
- added K_87: 4,15, josh-keyboard:MXOnly-1U-NoLED, F.Cu at (292.1, 109.5)
- added K_88: 4,16, josh-keyboard:MXOnly-1U-NoLED, F.Cu at (311.1, 109.5)
- added K_89: 4,18, josh-keyboard:MXOnly-2U-NoLED, F.Cu at (320.7, 109.5)
- added K_9: 0,7, josh-keyboard:MXOnly-1U-NoLED, F.Cu at (158.8, 33.3)
- added K_90: 5,4, josh-keyboard:MXOnly-1U-NoLED, F.Cu at (101.6, 128.6)
- added K_91: 5,13, josh-keyboard:MXOnly-1U-NoLED, F.Cu at (254.0, 128.6)
- added K_92: 5,0, josh-keyboard:MXOnly-1U-NoLED, F.Cu at (25.4, 128.6)
- added K_93: 5,1, josh-keyboard:MXOnly-1U-NoLED, F.Cu at (44.5, 128.6)
- added K_94: 5,2, josh-keyboard:MXOnly-1U-NoLED, F.Cu at (63.5, 128.6)
- added K_95: 5,3, josh-keyboard:MXOnly-1U-NoLED, F.Cu at (82.5, 128.6)
- added K_96: 5,5, josh-keyboard:MXOnly-3U-ReversedStabilizers-NoLED, F.Cu at (101.6, 128.6)
- added K_97: 5,6, josh-keyboard:MXOnly-1U-NoLED, F.Cu at (120.7, 128.6)
- added K_98: 5,7, josh-keyboard:MXOnly-1U-NoLED, F.Cu at (139.7, 128.6)
- added K_99: 5,8, josh-keyboard:MXOnly-1U-NoLED, F.Cu at (158.8, 128.6)
- added Q1: BSS138, Package_TO_SOT_SMD:SOT-23, B.Cu at (76.2, 42.9)
- added Q2: DTC123J, DTC123JKAT146:SOT95P280X100-3N, B.Cu at (38.1, 58.7)
- added R1: 10K, Resistor_SMD:R_0603_1608Metric, B.Cu at (76.2, 45.6)
- added R2: 10K, Resistor_SMD:R_0603_1608Metric, B.Cu at (78.9, 42.9)
- added R3: 5k1, Resistor_SMD:R_0603_1608Metric, B.Cu at (30.2, 54.8)
- added R4: 5k1, Resistor_SMD:R_0603_1608Metric, B.Cu at (30.2, 56.4)
- added R5: 1K5, Resistor_SMD:R_0603_1608Metric, B.Cu at (101.3, 77.6)
- added R6: 5K1, Resistor_SMD:R_0603_1608Metric, B.Cu at (15.9, 44.5)
- added R7: 100K, Resistor_SMD:R_0603_1608Metric, B.Cu at (35.7, 64.3)
- added SW1: EVQPUL02K, josh-buttons-switches:Panasonic_EVQPUL_EVQPUC, B.Cu at (15.9, 38.1)
- added U1: AP2112K-3.3, Package_TO_SOT_SMD:SOT-23-5, B.Cu at (92.1, 61.9)
- added U2: USBLC6-2SC6, Package_TO_SOT_SMD:SOT-23-6, B.Cu at (17.5, 52.4)
- added U3: STM32F303RCTx, Package_QFP:LQFP-64_10x10mm_P0.5mm, B.Cu at (110.5, 79.2)
- added Yw: 8MHz, josh-oscillators:Crystal_SMD_3225-4Pin_3.2x2.5mm, B.Cu at (121.2, 80.0)
Other:
- board outline added: 336.5 x 120.7 mm
- net class Default: via_dia 0.8 -> 0.6; via_drill 0.4 -> 0.3
